File: ripple-carry-adder.kicad_sch (KiCad schematic)
At the start: 20 parts, among them SW1 SW_DIP_x08

Commit message: new plaque
Other:
- company: Abteilung Biomed/Informatik -> Abteilung ELIT
Changed lines of the file:
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@@
 	(title_block
 		(title "4bit Ripple Carry Adder")
-		(date "Datum")
+		(date "2026-09-29")
 		(rev "V1.0 / R1")
-		(company "Abteilung Biomed/Informatik")
-		(comment 1 "Name")
-		(comment 2 "Klasse")
-		(comment 3 "gez")
-		(comment 4 "gepr")
-		(comment 5 "Betr")
+		(company "Abteilung ELIT")
+		(comment 1 "AndF JunJ ObeM SinS")
+		(comment 2 "3AHELS")
+		(comment 3 "AndF")
+		(comment 4 "SalH")
+		(comment 5 "HauP")
 		(comment 6 "Schematic")
 		(comment 8 "Prototyp")
